File: hw2/Arduino.sch (KiCad schematic (older format))
At the start: 28 parts, among them P1 CONN_01X02, P2 CONN_01X12, P3 CONN_01X12, U1 MIC5219, U2 ATmega32U4

Commit message: USB footprint correctd; routing updated; report updated
Parts:
- CONN1: footprint (none) -> Connectors:USB_Micro-B
Changed lines of the file:
@@
 $EndComp
 $Comp
-L GND #PWR5
+L GND #PWR01
 U 1 1 58A35B7E
 P 3450 2000
-F 0 "#PWR5" H 3450 1750 50  0001 C CNN
+F 0 "#PWR01" H 3450 1750 50  0001 C CNN
 F 1 "GND" H 3450 1850 50  0000 C CNN
 F 2 "" H 3450 2000 50  0000 C CNN
@@
 $EndComp
 $Comp
-L GND #PWR6
+L GND #PWR02
 U 1 1 58A35BAD
 P 3850 2000
-F 0 "#PWR6" H 3850 1750 50  0001 C CNN
+F 0 "#PWR02" H 3850 1750 50  0001 C CNN
 F 1 "GND" H 3850 1850 50  0000 C CNN
 F 2 "" H 3850 2000 50  0000 C CNN
@@
 $EndComp
 $Comp
-L GND #PWR7
+L GND #PWR03
 U 1 1 58A35BDC
 P 4150 2000
-F 0 "#PWR7" H 4150 1750 50  0001 C CNN
+F 0 "#PWR03" H 4150 1750 50  0001 C CNN
 F 1 "GND" H 4150 1850 50  0000 C CNN
 F 2 "" H 4150 2000 50  0000 C CNN
@@
 NoConn ~ 3000 1900
 $Comp
-L GND #PWR10
+L GND #PWR04
 U 1 1 58A35CC6
 P 4900 2350
-F 0 "#PWR10" H 4900 2100 50  0001 C CNN
+F 0 "#PWR04" H 4900 2100 50  0001 C CNN
 F 1 "GND" H 4900 2200 50  0000 C CNN
 F 2 "" H 4900 2350 50  0000 C CNN
@@
 $EndComp
 $Comp
-L GND #PWR2
+L GND #PWR05
 U 1 1 58A35D47
 P 1450 2100
-F 0 "#PWR2" H 1450 1850 50  0001 C CNN
+F 0 "#PWR05" H 1450 1850 50  0001 C CNN
 F 1 "GND" H 1450 1950 50  0000 C CNN
 F 2 "" H 1450 2100 50  0000 C CNN
@@
 $EndComp
 $Comp
-L GND #PWR4
+L GND #PWR06
 U 1 1 58A35D76
 P 1950 2100
-F 0 "#PWR4" H 1950 1850 50  0001 C CNN
+F 0 "#PWR06" H 1950 1850 50  0001 C CNN
 F 1 "GND" H 1950 1950 50  0000 C CNN
 F 2 "" H 1950 2100 50  0000 C CNN
@@
 $EndComp
 $Comp
-L VCC #PWR9
+L VCC #PWR07
 U 1 1 58A35EC2
 P 4900 1300
-F 0 "#PWR9" H 4900 1150 50  0001 C CNN
+F 0 "#PWR07" H 4900 1150 50  0001 C CNN
 F 1 "VCC" H 4900 1450 50  0000 C CNN
 F 2 "" H 4900 1300 50  0000 C CNN
@@
 $EndComp
 $Comp
-L GND #PWR11
+L GND #PWR08
 U 1 1 58A385E3
 P 4900 3800
-F 0 "#PWR11" H 4900 3550 50  0001 C CNN
+F 0 "#PWR08" H 4900 3550 50  0001 C CNN
 F 1 "GND" H 4900 3650 50  0000 C CNN
 F 2 "" H 4900 3800 50  0000 C CNN
@@
 $EndComp
 $Comp
-L GND #PWR13
+L GND #PWR09
 U 1 1 58A38627
 P 5900 2900
-F 0 "#PWR13" H 5900 2650 50  0001 C CNN
+F 0 "#PWR09" H 5900 2650 50  0001 C CNN
 F 1 "GND" H 5900 2750 50  0000 C CNN
 F 2 "" H 5900 2900 50  0000 C CNN
@@
 $EndComp
 $Comp
-L GND #PWR12
+L GND #PWR010
 U 1 1 58A3868B
 P 5500 3950
-F 0 "#PWR12" H 5500 3700 50  0001 C CNN
+F 0 "#PWR010" H 5500 3700 50  0001 C CNN
 F 1 "GND" H 5500 3800 50  0000 C CNN
 F 2 "" H 5500 3950 50  0000 C CNN
@@
 $EndComp
 $Comp
-L GND #PWR14
+L GND #PWR011
 U 1 1 58A386CF
 P 5900 3850
-F 0 "#PWR14" H 5900 3600 50  0001 C CNN
+F 0 "#PWR011" H 5900 3600 50  0001 C CNN
 F 1 "GND" H 5900 3700 50  0000 C CNN
 F 2 "" H 5900 3850 50  0000 C CNN
@@
 $EndComp
 $Comp
-L VCC #PWR16
+L VCC #PWR012
 U 1 1 58A38733
 P 6400 1150
-F 0 "#PWR16" H 6400 1000 50  0001 C CNN
+F 0 "#PWR012" H 6400 1000 50  0001 C CNN
 F 1 "VCC" H 6400 1300 50  0000 C CNN
 F 2 "" H 6400 1150 50  0000 C CNN
@@
 $EndComp
 $Comp
-L VCC #PWR17
+L VCC #PWR013
 U 1 1 58A38797
 P 6750 1300
-F 0 "#PWR17" H 6750 1150 50  0001 C CNN
+F 0 "#PWR013" H 6750 1150 50  0001 C CNN
 F 1 "VCC" H 6750 1450 50  0000 C CNN
 F 2 "" H 6750 1300 50  0000 C CNN
@@
 $EndComp
 $Comp
-L GND #PWR18
+L GND #PWR014
 U 1 1 58A38EE5
 P 6750 4800
-F 0 "#PWR18" H 6750 4550 50  0001 C CNN
+F 0 "#PWR014" H 6750 4550 50  0001 C CNN
 F 1 "GND" H 6750 4650 50  0000 C CNN
 F 2 "" H 6750 4800 50  0000 C CNN
@@
 $EndComp
 $Comp
-L GND #PWR20
+L GND #PWR015
 U 1 1 58A39270
 P 9750 4150
-F 0 "#PWR20" H 9750 3900 50  0001 C CNN
+F 0 "#PWR015" H 9750 3900 50  0001 C CNN
 F 1 "GND" H 9750 4000 50  0000 C CNN
 F 2 "" H 9750 4150 50  0000 C CNN
@@
 $EndComp
 $Comp
-L VCC #PWR22
+L VCC #PWR016
 U 1 1 58A3971C
 P 10700 3550
-F 0 "#PWR22" H 10700 3400 50  0001 C CNN
+F 0 "#PWR016" H 10700 3400 50  0001 C CNN
 F 1 "VCC" H 10700 3700 50  0000 C CNN
 F 2 "" H 10700 3550 50  0000 C CNN
@@
 $EndComp
 $Comp
-L VCC #PWR21
+L VCC #PWR017
 U 1 1 58A3976C
 P 10700 3250
-F 0 "#PWR21" H 10700 3100 50  0001 C CNN
+F 0 "#PWR017" H 10700 3100 50  0001 C CNN
 F 1 "VCC" H 10700 3400 50  0000 C CNN
 F 2 "" H 10700 3250 50  0000 C CNN
@@
 $EndComp
 $Comp
-L GND #PWR8
+L GND #PWR018
 U 1 1 58A3CA70
 P 4850 4750
-F 0 "#PWR8" H 4850 4500 50  0001 C CNN
+F 0 "#PWR018" H 4850 4500 50  0001 C CNN
 F 1 "GND" H 4850 4600 50  0000 C CNN
 F 2 "" H 4850 4750 50  0000 C CNN
@@
 	6850 2900 6850 3000
 $Comp
-L GND #PWR19
+L GND #PWR019
 U 1 1 58A4E3D9
 P 6850 3000
-F 0 "#PWR19" H 6850 2750 50  0001 C CNN
+F 0 "#PWR019" H 6850 2750 50  0001 C CNN
 F 1 "GND" H 6850 2850 50  0000 C CNN
 F 2 "" H 6850 3000 50  0000 C CNN
@@
 NoConn ~ 2650 5150
 $Comp
-L VCC #PWR15
+L VCC #PWR020
 U 1 1 58A65E09
 P 5900 5550
-F 0 "#PWR15" H 5900 5400 50  0001 C CNN
+F 0 "#PWR020" H 5900 5400 50  0001 C CNN
 F 1 "VCC" H 5900 5700 50  0000 C CNN
 F 2 "" H 5900 5550 50  0000 C CNN
@@
 $EndComp
 $Comp
-L VCC #PWR3
+L VCC #PWR021
 U 1 1 58A64122
 P 1500 2900
-F 0 "#PWR3" H 1500 2750 50  0001 C CNN
+F 0 "#PWR021" H 1500 2750 50  0001 C CNN
 F 1 "VCC" H 1500 3050 50  0000 C CNN
 F 2 "" H 1500 2900 50  0000 C CNN
@@
 $EndComp
 $Comp
-L PWR_FLAG #FLG2
+L PWR_FLAG #FLG022
 U 1 1 58A6418A
 P 2500 4550
-F 0 "#FLG2" H 2500 4645 50  0001 C CNN
+F 0 "#FLG022" H 2500 4645 50  0001 C CNN
 F 1 "PWR_FLAG" H 2500 4730 50  0000 C CNN
 F 2 "" H 2500 4550 50  0000 C CNN
@@
 $EndComp
 $Comp
-L PWR_FLAG #FLG1
+L PWR_FLAG #FLG023
 U 1 1 58A641F2
 P 1000 3000
-F 0 "#FLG1" H 1000 3095 50  0001 C CNN
+F 0 "#FLG023" H 1000 3095 50  0001 C CNN
 F 1 "PWR_FLAG" H 1000 3180 50  0000 C CNN
 F 2 "" H 1000 3000 50  0000 C CNN
@@
 $EndComp
 $Comp
-L GND #PWR1
+L GND #PWR024
 U 1 1 58A6425A
 P 1100 2900
-F 0 "#PWR1" H 1100 2650 50  0001 C CNN
+F 0 "#PWR024" H 1100 2650 50  0001 C CNN
 F 1 "GND" H 1100 2750 50  0000 C CNN
 F 2 "" H 1100 2900 50  0000 C CNN
@@
 F 0 "CONN1" H 3950 6750 60  0000 C CNN
 F 1 "MICRO_USB" H 4000 5950 60  0000 C CNN
-F 2 "" H 3950 6350 60  0000 C CNN
+F 2 "Connectors:USB_Micro-B" H 3950 6350 60  0001 C CNN
 F 3 "" H 3950 6350 60  0000 C CNN
 	1    3950 6350
